File: bigp4ppa.sch (KiCad schematic (older format))
At the start: 21 parts, among them J1 Power Input, J11 VOLTAGE19, J12 VOLTAGE12, J13 VOLTAGE13, J14 VOLTAGE18, J15 ADXL345, J2 Raspberry_Pi, J3 VOLTAGEFAN, J4 Output, J8 MAX13865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

Commit message: notes, pics, sample config
Parts:
- J1: footprint !Greg:TerminalBlock_TE_282834-4_1x04_P2.54mm_Horizontal -> !custom:TerminalBlock_TE_282834-4_1x04_P2.54mm_Horizontal
Changed lines of the file:
@@
 F 0 "J1" H 718 775 50  0000 C CNN
 F 1 "Power Input" H 718 866 50  0000 C CNN
-F 2 "!Greg:TerminalBlock_TE_282834-4_1x04_P2.54mm_Horizontal" H 800 1200 50  0001 C CNN
+F 2 "!custom:TerminalBlock_TE_282834-4_1x04_P2.54mm_Horizontal" H 800 1200 50  0001 C CNN
 F 3 "~" H 800 1200 50  0001 C CNN
 	1    800  1200
